Commit message: Added gps odometry, started on high resolution mapping, many other changes to get working.

File: config/robot.urdf.xacro (robot description, xacro)
@@ -2,34 +2,34 @@
 <robot name="lio" xmlns:xacro="http://tixiaoshan.github.io/">
   <xacro:property name="PI" value="3.1415926535897931" />
+  <link name="base_link"></link>
   <link name="chassis_link"></link>
-  <link name="base_link"></link>
-  <joint name="base_link_joint" type="fixed">
+  <joint name="chassis_joint" type="fixed">
     <parent link="base_link"/>
     <child link="chassis_link" />
     <origin xyz="0 0 0" rpy="0 0 0" />
   </joint>
-  <link name="lidar_link"> </link>
-  <joint name="lidar_joint" type="fixed">
-    <parent link="base_link" />
-    <child link="lidar_link" />
+  <link name="os_sensor"> </link>
+  <joint name="os_joint" type="fixed">
+    <parent link="chassis_link" />
+    <child link="os_sensor" />
     <origin xyz="0 0 0" rpy="0 0 0" />
   </joint>
-  <link name="imu_link"> </link>
+  <link name="imu"> </link>
   <joint name="imu_joint" type="fixed">
     <parent link="chassis_link" />
-    <child link="imu_link" />
-    <origin xyz="0 0 0" rpy="0 0 0" />
+    <child link="imu" />
+    <origin xyz="-0.085 0.0 -0.055" rpy="0 0 0" />
   </joint>
-  <link name="laser_sensor_frame"> </link>
-  <joint name="laser_joint" type="fixed">
-    <parent link="imu_link" />
-    <child link="laser_sensor_frame" />
-    <origin xyz="0 0 0" rpy="0 0 0" />
+  <link name="zed_camera_link"> </link>
+  <joint name="zed_joint" type="fixed">
+    <parent link="chassis_link" />
+    <child link="zed_camera_link" />
+    <origin xyz="0.0287 0 -0.0485" rpy="0 0 ${pi}" />
   </joint>
-  <link name="navsat_link"> </link>
-  <joint name="navsat_joint" type="fixed">
+  <link name="gps"> </link>
+  <joint name="gps_joint" type="fixed">
     <parent link="chassis_link" />
-    <child link="navsat_link" />
-    <origin xyz="0 0 0" rpy="0 0 0" />
+    <child link="gps" />
+    <origin xyz="-0.085 0.0 -0.055" rpy="0 0 0" />
   </joint>
 </robot>

Commit message: Changes during testing

File: config/robot.urdf.xacro (robot description, xacro)
@@ -19,10 +19,10 @@
     <parent link="chassis_link" />
     <child link="imu" />
-    <origin xyz="-0.085 0.0 -0.055" rpy="0 0 0" />
+    <origin xyz="0.0 0.0 -0.0946" rpy="0 0 0" />
   </joint>
-  <link name="zed_camera_link"> </link>
+  <link name="zed_camera_center"> </link>
   <joint name="zed_joint" type="fixed">
     <parent link="chassis_link" />
-    <child link="zed_camera_link" />
+    <child link="zed_camera_center" />
     <origin xyz="0.0287 0 -0.0485" rpy="0 0 ${pi}" />
   </joint>
@@ -31,5 +31,5 @@
     <parent link="chassis_link" />
     <child link="gps" />
-    <origin xyz="-0.085 0.0 -0.055" rpy="0 0 0" />
+    <origin xyz="0.0 0.0 -0.0946" rpy="0 0 0" />
   </joint>
 </robot>

Commit message: Work to get localistaion working, changed the imu update ratte to 150 from 500 in imuPre,  plus added PCL feature extraction which is a bit compute heavy...

File: config/robot.urdf.xacro (robot description, xacro)
@@ -19,11 +19,5 @@
     <parent link="chassis_link" />
     <child link="imu" />
-    <origin xyz="0.0 0.0 -0.0946" rpy="0 0 0" />
-  </joint>
-  <link name="zed_camera_center"> </link>
-  <joint name="zed_joint" type="fixed">
-    <parent link="chassis_link" />
-    <child link="zed_camera_center" />
-    <origin xyz="0.0287 0 -0.0485" rpy="0 0 ${pi}" />
+    <origin xyz="0.0 0.0 -0.0899" rpy="0 0 0" />
   </joint>
   <link name="gps"> </link>
@@ -31,5 +25,5 @@
     <parent link="chassis_link" />
     <child link="gps" />
-    <origin xyz="0.0 0.0 -0.0946" rpy="0 0 0" />
+    <origin xyz="0.0 0.0 -0.0899" rpy="0 0 0" />
   </joint>
 </robot>

Commit message: Some config changes, plus small changes to gps factor in mapOpt

File: config/robot.urdf.xacro (robot description, xacro)
@@ -7,5 +7,5 @@
     <parent link="base_link"/>
     <child link="chassis_link" />
-    <origin xyz="0 0 0" rpy="0 0 0" />
+    <origin xyz="0 0 0" rpy="0 ${0.0*PI/180.0} 0" />
   </joint>
   <link name="os_sensor"> </link>
@@ -19,5 +19,5 @@
     <parent link="chassis_link" />
     <child link="imu" />
-    <origin xyz="0.0 0.0 -0.0899" rpy="0 0 0" />
+    <origin xyz="0.0 0.0 -0.08011" rpy="0 0 0" />
   </joint>
   <link name="gps"> </link>
@@ -25,5 +25,5 @@
     <parent link="chassis_link" />
     <child link="gps" />
-    <origin xyz="0.0 0.0 -0.0899" rpy="0 0 0" />
+    <origin xyz="0.0 0.0 -0.08011" rpy="0 0 0" />
   </joint>
 </robot>

Commit message: Reverted to not using localisaiton nodes as was having issues with the LIO synchronising itselt to GPS..

File: config/robot.urdf.xacro (robot description, xacro)
@@ -7,5 +7,5 @@
     <parent link="base_link"/>
     <child link="chassis_link" />
-    <origin xyz="0 0 0" rpy="0 ${0.0*PI/180.0} 0" />
+    <origin xyz="0 0 0" rpy="0 0 0" />
   </joint>
   <link name="os_sensor"> </link>

Commit message: Config changes from Syslogic.

File: config/robot.urdf.xacro (robot description, xacro)
@@ -7,5 +7,5 @@
     <parent link="base_link"/>
     <child link="chassis_link" />
-    <origin xyz="0 0 0" rpy="0 0 0" />
+    <origin xyz="0 0 0" rpy="0 ${0.0*PI/180.0} 0" />
   </joint>
   <link name="os_sensor"> </link>
